File: Protogasm/ProtoPi-Board/ProtoPi-Board.kicad_sch (KiCad schematic)
At the start: 11 parts, among them J1 Neopixel_Ring_Header, J2 Jack-DC, M1 Motor_DC, Q1 FQP30N06L, SW1 Rotary_Encoder_Switch, U1 Arduino_UNO_R3, U2 MPX5050GP

Commit message: v5
Parts:
- removed U1: Arduino_UNO_R3, Module:Arduino_UNO_R3_WithMountingHoles, symbol MCU_Module:Arduino_UNO_R3
- added C2, C3: 10u, Capacitor_THT:CP_Radial_D5.0mm_P2.50mm, symbol Device:C_Polarized_US
- added J3: Raspberry_Pi_2_3, custom-footprints:Raspberry_Pi_4_Model_B, symbol Connector:Raspberry_Pi_2_3
- added R3: 2k, Resistor_THT:R_Axial_DIN0207_L6.3mm_D2.5mm_P7.62mm_Horizontal, symbol Device:R_US
- added SW2: FOOTSWITCH, custom-footprints:Motor_DC_WirePins, symbol Switch:SW_SPST
- added SW3: (no value), symbol Switch:SW_SPST
- added U1: R-78E5.0-0.5, Converter_DCDC:Converter_DCDC_RECOM_R-78E-0.5_THT, symbol Regulator_Switching:R-78E5.0-0.5
- added U3: TXB0108, custom-footprints:TXB0108-Adafruit, symbol Logic_LevelTranslator:TXB0108DQSR
- added U4: MCP3008, Package_DIP:DIP-16_W7.62mm, symbol Analog_ADC:MCP3008
Connections:
- net +12V: now also C2.1, U1.1 (IN)
- net +5V: now also C3.1, U1.3 (OUT), U3.20 (VCCB), U4.16 (Vdd)
- net GND: now also C2.2, C3.2, J3.6 (GND), SW2.2 (B), SW3.2 (B), U1.2 (GND), U3.11 (GND), U4.14 (AGND), U4.9 (DGND)
- net A0 renamed A_CH0
- net A_CH0: now also U4.1 (CH0)
- net AREF renamed A_REF
- net A_REF: now also U4.15 (Vref)
- net D10 renamed NEO_DATA_5V
- net NEO_DATA_5V: now also U3.15 (B5)
- net D2 renamed SW_ROTA
- net SW_ROTA: now also J3.8 (GPIO14/TXD)
- net D3 renamed SW_ROTB
- net SW_ROTB: now also J3.10 (GPIO15/RXD)
- net D5 renamed SW_PRESS
- net SW_PRESS: now also J3.36 (GPIO16)
- net D9 renamed MOTOR_3V3
- net MOTOR_3V3: now also J3.12 (GPIO18/PWM0)
- new net: J3.27 (ID_SD/GPIO0), R3.2, SW2.1 (A), SW3.1 (A)
- new net +3V3: J3.1 (3V3), R3.1, U3.1 (VCCA)
- new net CLK_3V3: J3.23 (SCLK0/GPIO11), U3.2 (A1)
- new net CLK_5V: U3.19 (B1), U4.13 (CLK)
- new net MISO_3V3: J3.21 (MISO0/GPIO9), U3.3 (A2)
- new net MISO_5V: U3.18 (B2), U4.12 (Dout)
- new net MOSI_3V3: J3.19 (MOSI0/GPIO10), U3.4 (A3)
- new net MOSI_5V: U3.17 (B3), U4.11 (Din)
- new net NEO_DATA_3V3: J3.40 (GPIO21/SCLK1), U3.6 (A5)
- new net TXB_OE: J3.31 (GCLK2/GPIO6), U3.10 (OE)
- new net ~{CS_3V3}: J3.13 (GPIO27), U3.5 (A4)
- new net ~{CS_5V}: U3.16 (B4), U4.10 (~{CS}/SHDN)
- no-connect marks 25 -> 43
Other:
- title: Protogasm -> ProtoPi
- moved on the sheet: C1, D1, J1, J2, M1, Q1, R1, R2, SW1, U2
